File: HamShieldMini1.2.kicad_pcb (KiCad board)
At the start: 4 copper layers, 65 x 30 mm, 200 parts, among them J1 SMA_EDGE, J2 SJ-43514-SMT-TR, P1 Conn_01x10, P2 Conn_01x07, Q1 NTGD1100L, Q5 BSS138, Q6 BSS138, Q7 BSS138, U1 AU1846, U10 PE42440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

Commit message: unify pin naming scheme
Connections:
- net /SCLK renamed /CLK
- net /SDIO renamed /DAT
- net /nSEN renamed /nCS
- U1 pad 10: Net-(U1-Pad10) -> (no net)
- U1 pad 14: Net-(U1-Pad14) -> (no net)
- U1 pad 17: Net-(U1-Pad17) -> (no net)
- U1 pad 19: Net-(U1-Pad19) -> (no net)
- U1 pad 20: Net-(U1-Pad20) -> (no net)
- U1 pad 22: Net-(U1-Pad22) -> (no net)
- U11 pad 12: Net-(U11-Pad12) -> (no net)
- U12 pad 6: /Y2 -> (no net)
