File: HamShieldMini1.2.sch (KiCad schematic (older format))
At the start: 25 parts, among them P1 Conn_01x10, U1 AU1846, U12 NC7WZ14, Y1 12.8MHz

Commit message: unify pin naming scheme
Connections:
- net labels added: CLK, DAT, nCS
- net labels removed: SCLK, SDIO, nSEN
Changed lines of the file:
@@
 F0 "User Interface" 60
 F1 "UserInterface.sch" 60
-F2 "SCLK" O L 1500 2050 60
-F3 "SDIO" B L 1500 1900 60
+F2 "CLK" O L 1500 2050 60
+F3 "DAT" B L 1500 1900 60
 F4 "PDN" O R 2700 850 60
 F5 "AFOUT" I L 1500 850 60
 F6 "MIC_IN" O L 1500 1000 60
-F7 "nSEN" I L 1500 1750 60
+F7 "nCS" I L 1500 1750 60
 F8 "MODE" I L 1500 1600 60
 $EndSheet
@@
 PDN
 Text Label 2500 3300 0    60   ~ 0
-SCLK
+CLK
 Text Label 2500 3550 0    60   ~ 0
-SDIO
+DAT
 Text Label 750  2050 0    60   ~ 0
-SCLK
+CLK
 Text Label 750  1900 0    60   ~ 0
-SDIO
+DAT
 Wire Wire Line
 	5800 900  5800 2350
@@
 	2950 4550 3400 4550
 Text Label 2950 4800 0    60   ~ 0
-nSEN
+nCS
 Wire Wire Line
 	1500 1750 750  1750
 Text Label 750  1750 0    60   ~ 0
-nSEN
+nCS
 Text Label 2950 4550 0    60   ~ 0
 MODE
