File: UserInterface.sch (KiCad schematic (older format))
At the start: 38 parts, among them J2 SJ-43514-SMT-TR, P2 Conn_01x07, Q5 BSS138, Q6 BSS138, Q7 BSS138, U3 AD8591

Commit message: unify pin naming scheme
Connections:
- net labels added: CLK, DAT, nCS
- net labels removed: SCLK, SDIO, nSEN
Changed lines of the file:
@@
 AFOUT
 Text HLabel 1050 2900 0    60   Input ~ 0
-SCLK
+CLK
 Text HLabel 1050 2450 0    60   Input ~ 0
-SDIO
+DAT
 Text HLabel 1050 7550 2    60   Input ~ 0
 PDN
@@
 $EndComp
 Text HLabel 1050 2000 0    60   Input ~ 0
-nSEN
+nCS
 $Comp
 L power:VCC #PWR086
